File: SoundLazer/SoundLazer.sch (KiCad schematic (older format))
At the start: 115 parts, among them J1 Audio_in, J2 DSP_PROG, J3 PWR_SEL, J4 12V_IN, J5 SPK_OUT, Q1 ZXTP25040DZTA, Q2 MMDT2222V, Q3 MMDT2907V, Q4 FDS4935A, Q5 FDS6890A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

Commit message: first revision
Parts:
- added R32, R33: 10k, Resistor_SMD:R_0402_1005Metric, symbol Device:R
- added TP4: Audio_out, TestPoint:TestPoint_THTPad_D1.5mm_Drill0.7mm, symbol Connector:TestPoint
- added unit 4 of U3
- added unit 5 of U3
- added unit 6 of U3
- R16: value 56.2k -> 1k
- R17: value 49.9k -> 3.32k
Connections:
- net DSP_A_OUT: now also TP4.1
- net GND: now also R32.1, R33.1, U3.11, U3.14, U3.9
- net ~RST: now also R33.2
- net at TP1.1, U2.10 (E2), U3.3: now also R32.2
Changed lines of the file:
@@
 U 1 1 60ADEA2A
 P 10000 10200
-F 0 "R27" V 9793 10200 50  0000 C CNN
+F 0 "R27" V 9950 10000 50  0000 C CNN
 F 1 "10" V 9884 10200 50  0000 C CNN
 F 2 "Resistor_SMD:R_0402_1005Metric" V 9930 10200 50  0001 C CNN
@@
 U 1 1 60AE68C3
 P 10000 8350
-F 0 "R26" V 9793 8350 50  0000 C CNN
+F 0 "R26" V 9950 8100 50  0000 C CNN
 F 1 "10" V 9884 8350 50  0000 C CNN
 F 2 "Resistor_SMD:R_0402_1005Metric" V 9930 8350 50  0001 C CNN
@@
 P 6950 4100
 F 0 "R17" H 6880 4054 50  0000 R CNN
-F 1 "49.9k" H 6880 4145 50  0000 R CNN
+F 1 "3.32k" H 6880 4145 50  0000 R CNN
 F 2 "Resistor_SMD:R_0402_1005Metric" V 6880 4100 50  0001 C CNN
 F 3 "~" H 6950 4100 50  0001 C CNN
@@
 P 6850 1900
 F 0 "R16" H 6780 1854 50  0000 R CNN
-F 1 "56.2k" H 6780 1945 50  0000 R CNN
+F 1 "1k" H 6780 1945 50  0000 R CNN
 F 2 "Resistor_SMD:R_0402_1005Metric" V 6780 1900 50  0001 C CNN
 F 3 "~" H 6850 1900 50  0001 C CNN
@@
 DSP_A_OUT
 Wire Wire Line
-	9900 2500 9400 2500
+	10050 2500 9400 2500
 $Comp
 L power:+3V3 #PWR014
@@
 	14700 3750 14700 3800
 Wire Wire Line
-	14600 4250 14950 4250
+	14600 4250 15100 4250
 Wire Wire Line
 	13400 4250 13800 4250
@@
 Text Label 3750 5400 0    50   ~ 0
 ~MAN_RES
+$Comp
+L Device:R R33
+U 1 1 60BF57D4
+P 15100 4400
+F 0 "R33" H 15030 4354 50  0000 R CNN
+F 1 "10k" H 15030 4445 50  0000 R CNN
+F 2 "Resistor_SMD:R_0402_1005Metric" V 15030 4400 50  0001 C CNN
+F 3 "~" H 15100 4400 50  0001 C CNN
+	1    15100 4400
+	-1   0    0    1
+$EndComp
+$Comp
+L power:GND #PWR0102
+U 1 1 60BF624A
+P 15100 4550
+F 0 "#PWR0102" H 15100 4300 50  0001 C CNN
+F 1 "GND" H 15105 4377 50  0000 C CNN
+F 2 "" H 15100 4550 50  0001 C CNN
+F 3 "" H 15100 4550 50  0001 C CNN
+	1    15100 4550
+	1    0    0    -1
+$EndComp
+$Comp
+L Connector:TestPoint TP4
+U 1 1 60C1542B
+P 10050 2500
+F 0 "TP4" H 10108 2618 50  0000 L CNN
+F 1 "Audio_out" H 10108 2527 50  0000 L CNN
+F 2 "TestPoint:TestPoint_THTPad_D1.5mm_Drill0.7mm" H 10250 2500 50  0001 C CNN
+F 3 "~" H 10250 2500 50  0001 C CNN
+	1    10050 2500
+	1    0    0    -1
+$EndComp
+$Comp
+L Device:R R32
+U 1 1 60C55770
+P 4050 9500
+F 0 "R32" H 3980 9454 50  0000 R CNN
+F 1 "10k" H 3980 9545 50  0000 R CNN
+F 2 "Resistor_SMD:R_0402_1005Metric" V 3980 9500 50  0001 C CNN
+F 3 "~" H 4050 9500 50  0001 C CNN
+	1    4050 9500
+	-1   0    0    1
+$EndComp
+$Comp
+L power:GND #PWR0100
+U 1 1 60C55786
+P 4050 9650
+F 0 "#PWR0100" H 4050 9400 50  0001 C CNN
+F 1 "GND" H 4055 9477 50  0000 C CNN
+F 2 "" H 4050 9650 50  0001 C CNN
+F 3 "" H 4050 9650 50  0001 C CNN
+	1    4050 9650
+	1    0    0    -1
+$EndComp
+Wire Wire Line
+	4050 9350 4050 9300
+$Comp
+L 4xxx:4049 U3
+U 4 1 60C97B46
+P 6800 10300
+F 0 "U3" H 6800 10617 50  0000 C CNN
+F 1 "4049" H 6800 10526 50  0000 C CNN
+F 2 "" H 6800 10300 50  0001 C CNN
+F 3 "http://www.intersil.com/content/dam/intersil/documents/cd40/cd4049ubms.pdf" H 6800 10300 50  0001 C CNN
+	4    6800 10300
+	1    0    0    -1
+$EndComp
+$Comp
+L 4xxx:4049 U3
+U 5 1 60C99B06
+P 6800 10600
+F 0 "U3" H 7200 10500 50  0000 C CNN
+F 1 "4049" H 7000 10500 50  0000 C CNN
+F 2 "" H 6800 10600 50  0001 C CNN
+F 3 "http://www.intersil.com/content/dam/intersil/documents/cd40/cd4049ubms.pdf" H 6800 10600 50  0001 C CNN
+	5    6800 10600
+	1    0    0    -1
+$EndComp
+$Comp
+L 4xxx:4049 U3
+U 6 1 60C9B7E2
+P 6800 10900
+F 0 "U3" H 6800 10650 50  0000 C CNN
+F 1 "4049" H 6850 10750 50  0000 C CNN
+F 2 "" H 6800 10900 50  0001 C CNN
+F 3 "http://www.intersil.com/content/dam/intersil/documents/cd40/cd4049ubms.pdf" H 6800 10900 50  0001 C CNN
+	6    6800 10900
+	1    0    0    -1
+$EndComp
+$Comp
+L power:GND #PWR0101
+U 1 1 60CBBC61
+P 6500 10950
+F 0 "#PWR0101" H 6500 10700 50  0001 C CNN
+F 1 "GND" H 6505 10777 50  0000 C CNN
+F 2 "" H 6500 10950 50  0001 C CNN
+F 3 "" H 6500 10950 50  0001 C CNN
+	1    6500 10950
+	1    0    0    -1
+$EndComp
+Wire Wire Line
+	6500 10950 6500 10900
+Connection ~ 6500 10600
+Wire Wire Line
+	6500 10600 6500 10300
+Connection ~ 6500 10900
+Wire Wire Line
+	6500 10900 6500 10600
 $EndSCHEMATC

Commit message: r20 corr
Parts:
- R20: value 56.2k -> 56.2
Changed lines of the file:
@@
 P 8250 2500
 F 0 "R20" V 8150 2400 50  0000 R CNN
-F 1 "56.2k" V 8200 2800 50  0000 R CNN
+F 1 "56.2" V 8200 2800 50  0000 R CNN
 F 2 "Resistor_SMD:R_0402_1005Metric" V 8180 2500 50  0001 C CNN
 F 3 "~" H 8250 2500 50  0001 C CNN

Commit message: pcb update
Parts:
- removed C39: 220u 35V, Capacitor_SMD:C_Elec_8x10.2, symbol Device:CP
- removed J1: Audio_in, symbol Connector:AudioJack2_Ground
- added D4: LL-R3528RGBM, LED_SMD:LED_Avago_PLCC4_3.2x2.8mm_CW, symbol Device:LED_ARGB
- added H1, H2, H3, H4: M2.5, MountingHole:MountingHole_2.7mm_M2.5, symbol Mechanical:MountingHole
- added J1: Audio_in, Connector_Audio:Jack_3.5mm_Ledino_KB3SPRS_Horizontal, symbol Connector:AudioJack2_Ground_Switch
- added Q6, Q7, Q8: 2N7002, Package_TO_SOT_SMD:SOT-23, symbol Transistor_FET:2N7002
- added R34, R35, R36: 3.32k, Resistor_SMD:R_0402_1005Metric, symbol Device:R
- added R37, R38, R39, R40: 10k, Resistor_SMD:R_0402_1005Metric, symbol Device:R
- added SW2: EG1381A, Button_Switch_SMD:SW_SP3T_PCM13, symbol Switch:SW_SP3T
- C1, C14, C15, C16, C17, C2, C20, C21, C22, C23, C24, C3, C32, C33, C34, C36, C41, C45, C46, C48, C49, C50, C51: footprint Capacitor_SMD:C_0603_1608Metric -> Capacitor_SMD:C_0402_1005Metric
- F1: footprint (none) -> Fuse:Fuse_1206_3216Metric
- U2: footprint (none) -> Package_SO:TSSOP-16_4.4x5mm_P0.65mm
- U3: value 4049 -> HEF4049BT,653; footprint (none) -> Package_SO:SOIC-16_3.9x9.9mm_P1.27mm
Connections:
- net +3V3: now also R37.1, R38.2, R39.2
- net +6V: now also D4.1 (A)
- net GND: now also U3.7, J1.G, Q6.2 (S), Q7.2 (S), Q8.2 (S), R40.1; no longer U3.14
- net at C38.2, Q3.3 (C), R27.2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: now also Q2.4 (E2); no longer Q2.1 (E1)
- net at C29.1, Q3.5 (B), R19.1: now also Q2.5 (B2); no longer Q2.2 (B1)
- net at C37.2, Q3.6 (C), R26.2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: now also Q2.1 (E1); no longer Q2.4 (E2)
- net at C28.1, Q3.2 (B), R18.1: now also Q2.2 (B1); no longer Q2.5 (B2)
- net at C29.2, R19.2: now also U3.15; no longer U3.6
- net at C28.2, R18.2: now also J3.4 (Pin_4), U3.2; no longer J3.2 (Pin_2), U3.4
- net at J3.3 (Pin_3): now also R15.2, U3.14
- net at U3.5: now also R32.2, TP1.1, U2.10 (E2); no longer U3.2
- net at U4.15 (MP6): now also R39.1, SW2.4
- net at U4.19 (MP11): now also Q8.1 (G)
- net at U4.26 (MP9): now also Q7.1 (G)
- net at U4.27 (MP8): now also Q6.1 (G)
- net at U4.8 (MP4): now also R37.2, SW2.1
- net at U4.9 (MP5): now also R38.1, SW2.2
- net at FB2.2: now also J1.T
- net at FB1.2: now also J1.S
- new net: U3.3, U3.4
- new net: Q6.3 (D), R34.1
- new net: D4.2 (RK), R34.2
- new net: Q7.3 (D), R35.1
- new net: D4.3 (GK), R35.2
- new net: Q8.3 (D), R36.1
- new net: D4.4 (BK), R36.2
- new net: R40.2, SW2.3
- now unconnected: J3.1 (Pin_1)
Other:
- moved on the sheet: C27, C30, C31, C34, J3, Q2A, Q2B, R17, U3A, U3B, U3C, U3F

Commit message: pcb_finish
Parts:
- removed J1: Audio_in, Connector_Audio:Jack_3.5mm_Ledino_KB3SPRS_Horizontal, symbol Connector:AudioJack2_Ground_Switch
- added J1: SJ1-3523N, temp_pcb_lib:CUI_SJ1-3523N, symbol SJ1-3523N:SJ1-3523N
Connections:
- net GND: now also J1.1
- net at FB1.2: now also J1.3
- net at FB2.2: now also J1.2
Other:
- moved on the sheet: C10, C12, C13, C15, C16, C18, C19, C2, C20, C21, C22, C23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
