File: SoundLazer/SoundLazer.kicad_pcb (KiCad board)
At the start: 2 copper layers, 91 x 55 mm, 133 parts, among them J1 Audio_in, J2 DSP_PROG, J3 PWR_SEL, J4 12V_IN, J5 SPK_OUT, Q1 ZXTP25040DZTA, Q2 MMDT2222V, Q3 MMDT2907V, Q4 FDS4935A, Q5 FDS6890A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

Commit message: pcb_finish
Parts:
- J1: value Audio_in -> SJ1-3523N; footprint Connector_Audio:Jack_3.5mm_Ledino_KB3SPRS_Horizontal -> temp_pcb_lib:CUI_SJ1-3523N
- moved J1 4.81 mm to (113.8, 100.2)
Routing:
- net Net-(FB1-Pad2): track 2.62 -> 11.6 mm
- net Net-(FB2-Pad2): track 16.7 -> 12.7 mm
- net Net-(C38-Pad2): track 31.8 -> 32.7 mm
- net +3V3: track 183.5 -> 184.3 mm
- net GND: vias 40 -> 97
